Commit message: create model joints, setup env

File: Model/robot.urdf (robot description, URDF)
Before this commit: robot onshape, 1 links, 0 joints
Links:
- removed link arduinomotor
- added link base, mass 1406.2088699182115761; collision mesh filename=package:///baseplate.stl; collision mesh filename=package:///motor.stl
- added link legjointconnector2, mass 33.700879238921558567; collision mesh filename=package:///legjointconnector2.stl; visual mesh filename=package:///legjointconnector2.stl
- added link legjointconnector2_2, mass 33.700879238921558567; collision mesh filename=package:///legjointconnector2.stl; visual mesh filename=package:///legjointconnector2.stl
- added link legjointconnector2_3, mass 33.700879238921558567; collision mesh filename=package:///legjointconnector2.stl; visual mesh filename=package:///legjointconnector2.stl
- added link legjointconnector2_4, mass 33.700879238921558567; collision mesh filename=package:///legjointconnector2.stl; visual mesh filename=package:///legjointconnector2.stl
- added link legjointconnector4, mass 114.5044662372232267; collision mesh filename=package:///legjointconnector4.stl; visual mesh filename=package:///legjointconnector4.stl
- added link legjointconnector4_2, mass 114.5044662372232267; collision mesh filename=package:///legjointconnector4.stl; visual mesh filename=package:///legjointconnector4.stl
- added link legjointconnector4_3, mass 114.5044662372232267; collision mesh filename=package:///legjointconnector4.stl; visual mesh filename=package:///legjointconnector4.stl
- added link legjointconnector4_4, mass 114.5044662372232267; collision mesh filename=package:///legjointconnector4.stl; visual mesh filename=package:///legjointconnector4.stl
- added link segment1, mass 188.73631876709129074; collision mesh filename=package:///legjointconnector1.stl; collision mesh filename=package:///motor.stl
- added link segment1_2, mass 188.73631876709129074; collision mesh filename=package:///legjointconnector1.stl; collision mesh filename=package:///motor.stl
- added link segment1inverse, mass 188.73631876709129074; collision mesh filename=package:///legjointconnector1.stl; collision mesh filename=package:///motor.stl
- added link segment1inverse_2, mass 188.73631876709129074; collision mesh filename=package:///legjointconnector1.stl; collision mesh filename=package:///motor.stl
- added link segment3, mass 415.11154881410027429; collision mesh filename=package:///legjointconnector3.stl; collision mesh filename=package:///motor.stl
- added link segment3_2, mass 415.11154881410027429; collision mesh filename=package:///legjointconnector3.stl; collision mesh filename=package:///motor.stl
- added link segment3_3, mass 415.11154881410027429; collision mesh filename=package:///legjointconnector3.stl; collision mesh filename=package:///motor.stl
- added link segment3_4, mass 415.11154881410027429; collision mesh filename=package:///legjointconnector3.stl; collision mesh filename=package:///motor.stl
Joints:
- added joint BL_J1: type revolute, parent base, child segment1, origin xyz=0.49783999999999972719 0 0 rpy=1.2212454284373163526e-15 8.2675113504355278044e-16 1.5707963403039673089, axis 0 0 1, limit lower=0 upper=6.283185307179586232 effort=1 velocity=20
- added joint BL_J2: type revolute, parent segment1, child legjointconnector2, origin xyz=-0.45577759999999978291 -0.27635200000000015308 -0.12700000000000022382 rpy=-1.57079632679489678 3.8061645123399012522e-16 -3.141592653589793116, axis 0 0 1, limit lower=0 upper=6.283185307179586232 effort=1 velocity=20
- added joint BL_J3: type revolute, parent legjointconnector2, child segment3, origin xyz=0.20990560000000013652 -0.25054560000000003495 0 rpy=-5.5681001479697635813e-16 3.0198503996277484511e-16 3.141592653589793116, axis 0 0 1, limit lower=0 upper=6.283185307179586232 effort=1 velocity=20
- added joint BL_J4: type revolute, parent segment3, child legjointconnector4, origin xyz=-1.1645024028449062481 0 2.2204460492503130808e-16 rpy=1.6661838092530166565e-15 -5.2010781123730119761e-16 7.9619013065275774349e-18, axis 0 0 1, limit lower=0 upper=6.283185307179586232 effort=1 velocity=20
- added joint BR_J1: type revolute, parent base, child segment1inverse_2, origin xyz=0.49783999999999972719 0.9651999999999995028 0 rpy=1.7764361321532213574e-23 1.1952881864215707969e-23 -1.57079632679489678, axis 0 0 1, limit lower=0 upper=6.283185307179586232 effort=1 velocity=20
- added joint BR_J2: type revolute, parent segment1inverse_2, child legjointconnector2_3, origin xyz=-0.45577759999999967189 0.27635200000000015308 -0.12700000000000000178 rpy=1.570796326794896336 1.1102231566283779189e-16 -3.141592653589793116, axis 0 0 1, limit lower=0 upper=6.283185307179586232 effort=1 velocity=20
- added joint BR_J3: type revolute, parent legjointconnector2_3, child segment3_3, origin xyz=0.20990560000000035856 0.25054559999999992392 0 rpy=-4.2376321053686627128e-24 2.0116180994100064909e-31 3.141592653589793116, axis 0 0 1, limit lower=0 upper=6.283185307179586232 effort=1 velocity=20
- added joint BR_J4: type revolute, parent segment3_3, child legjointconnector4_3, origin xyz=-1.1645024028449080244 0 -4.4408920985006261617e-16 rpy=-9.0442043540577272659e-17 -4.478155192180798781e-17 -2.5970077749655048884e-17, axis 0 0 1, limit lower=0 upper=6.283185307179586232 effort=1 velocity=20
- added joint FL_J1: type revolute, parent segment1inverse, child base, origin xyz=-0.57807399120160729566 -0.5988052311389459037 -0.77874950167232726006 rpy=-2.3872993578795250843e-08 3.8169197161100659601e-08 -1.5707963267948970021, axis 0 0 1, limit lower=0 upper=6.283185307179586232 effort=1 velocity=20
- added joint FL_J2: type revolute, parent segment1inverse, child legjointconnector2_4, origin xyz=-1.0338515942334769449 -0.32245322629145822813 -0.90574948024341750408 rpy=1.5707962886256991997 -2.3872993467772918602e-08 -3.1415926535897926719, axis 0 0 1, limit lower=0 upper=6.283185307179586232 effort=1 velocity=20
- added joint FL_J3: type revolute, parent legjointconnector2_4, child segment3_4, origin xyz=0.20990560000000035856 0.2505455999999998129 5.5511151231257827021e-17 rpy=4.2376321985735554229e-24 1.0729593300831567566e-17 3.141592653589793116, axis 0 0 1, limit lower=0 upper=6.283185307179586232 effort=1 velocity=20
- added joint FL_J4: type revolute, parent segment3_4, child legjointconnector4_4, origin xyz=-1.1645024028449064701 -1.1102230246251565404e-16 1.1102230246251565404e-16 rpy=-1.110222826101810144e-16 -1.1778011199458197558e-30 -1.5278887872991683262e-23, axis 0 0 1, limit lower=0 upper=6.3006385996995293297 effort=1 velocity=20
- added joint FR_J1: type revolute, parent base, child segment1_2, origin xyz=0 0.96519999999999961382 0 rpy=2.9004576563626872302e-15 1.013078515305890832e-15 -1.5707963267948972241, axis 0 0 1, limit lower=0 upper=6.283185307179586232 effort=1 velocity=20
- added joint FR_J2: type revolute, parent segment1_2, child legjointconnector2_2, origin xyz=-0.4557775999999997274 -0.27635199999999998655 -0.12699999999999977973 rpy=-1.5707963267948947816 5.8286706669016316343e-16 3.141592653589793116, axis 0 0 1, limit lower=0 upper=6.283185307179586232 effort=1 velocity=20
- added joint FR_J3: type revolute, parent legjointconnector2_2, child segment3_2, origin xyz=0.2099056000000000255 -0.25054559999999992392 -5.5511151231257827021e-17 rpy=5.5511156512876473097e-17 1.8316849040800762374e-31 3.141592653589793116, axis 0 0 1, limit lower=0 upper=6.283185307179586232 effort=1 velocity=20
- added joint FR_J4: type revolute, parent segment3_2, child legjointconnector4_2, origin xyz=-1.1645024028449086906 -1.1102230246251565404e-16 1.6653345369377348106e-16 rpy=1.605866653096347499e-15 -4.3247425860249348976e-18 -4.0123531872111090802e-17, axis 0 0 1, limit lower=0 upper=6.283185307179586232 effort=1 velocity=20

Commit message: initialize joints, set limits

File: Model/robot.urdf (robot description, URDF)
Before this commit: robot onshape, 17 links, 16 joints
Links:
- link base: mass 1406.2088699182115761 -> 1406.2088699182118035
- link legjointconnector2: mass 33.700879238921558567 -> 33.700879238921572778
- link legjointconnector2_2: mass 33.700879238921558567 -> 33.700879238921572778
- link legjointconnector2_3: mass 33.700879238921558567 -> 33.700879238921572778
- link legjointconnector2_4: mass 33.700879238921558567 -> 33.700879238921572778
- link legjointconnector4: mass 114.5044662372232267 -> 114.50446623722325512
- link legjointconnector4_2: mass 114.5044662372232267 -> 114.50446623722325512
- link legjointconnector4_3: mass 114.5044662372232267 -> 114.50446623722325512
- link legjointconnector4_4: mass 114.5044662372232267 -> 114.50446623722325512
Joints:
- joint BL_J1: limit lower=0 upper=6.283185307179586232 effort=1 velocity=20 -> lower=0 upper=0.87266462599716476678 effort=1 velocity=20; origin xyz=0.49783999999999972719 0 0 rpy=1.2212454284373163526e-15 8.2675113504355278044e-16 1.5707963403039673089 -> xyz=-0.67928361386142521727 -0.69208391498186450086 -0.14137123396112205587 rpy=4.1366065074091267764e-08 -1.5386514204730299893e-08 0.87266463153054429913
- joint BL_J2: limit lower=0 upper=6.283185307179586232 effort=1 velocity=20 -> lower=-0.52359877559829881566 upper=1.3962634015954635824 effort=1 velocity=20; origin xyz=-0.45577759999999978291 -0.27635200000000015308 -0.12700000000000022382 rpy=-1.57079632679489678 3.8061645123399012522e-16 -3.141592653589793116 -> xyz=-0.4557775999999992278 -0.27635200000000270659 -0.12700000000000088995 rpy=-1.5707963267949023312 0.52359877559829381966 3.1415926535897895633
- joint BL_J3: limit lower=0 upper=6.283185307179586232 effort=1 velocity=20 -> lower=-0.34906585039886589561 upper=1.0471975511965976313 effort=1 velocity=20; origin xyz=0.20990560000000013652 -0.25054560000000003495 0 rpy=-5.5681001479697635813e-16 3.0198503996277484511e-16 3.141592653589793116 -> xyz=0.20990559999999991447 -0.25054559999999986841 2.2204460492503130808e-16 rpy=-7.1969438406019748775e-14 3.7780358523688956078e-14 -3.1415926535897917837
- joint BL_J4: limit lower=0 upper=6.283185307179586232 effort=1 velocity=20 -> lower=-0.34906585039886589561 upper=1.0471975511965976313 effort=1 velocity=20; origin xyz=-1.1645024028449062481 0 2.2204460492503130808e-16 rpy=1.6661838092530166565e-15 -5.2010781123730119761e-16 7.9619013065275774349e-18 -> xyz=-1.1645024028448791586 3.3306690738754696213e-16 -3.7359004778636517585e-14 rpy=7.2159191514795347321e-14 -3.8605192353852867702e-14 9.6550876637817448444e-15
- joint BR_J1: limit lower=0 upper=6.283185307179586232 effort=1 velocity=20 -> lower=-0.87266462599716476678 upper=0 effort=1 velocity=20; origin xyz=0.49783999999999972719 0.9651999999999995028 0 rpy=1.7764361321532213574e-23 1.1952881864215707969e-23 -1.57079632679489678 -> xyz=-0.058865017083267592857 0.04730218494957370845 -0.14137121911005823272 rpy=-4.1366065085108797363e-08 1.5386514061235917372e-08 -2.2689280220592675796
- joint BR_J2: child legjointconnector2_3 -> legjointconnector2_4; limit lower=0 upper=6.283185307179586232 effort=1 velocity=20 -> lower=-1.3962634015954635824 upper=0.52359877559829881566 effort=1 velocity=20; origin xyz=-0.45577759999999967189 0.27635200000000015308 -0.12700000000000000178 rpy=1.570796326794896336 1.1102231566283779189e-16 -3.141592653589793116 -> xyz=-0.45577759999999967189 0.27635199999999970899 -0.12700000000000022382 rpy=1.5707963267948970021 0.52359877559830325655 -3.1415926535897926719
- joint BR_J3: child segment3_3 -> segment3_4; limit lower=0 upper=6.283185307179586232 effort=1 velocity=20 -> lower=-1.0471975511965976313 upper=0.34906585039886589561 effort=1 velocity=20; origin xyz=0.20990560000000035856 0.25054559999999992392 0 rpy=-4.2376321053686627128e-24 2.0116180994100064909e-31 3.141592653589793116 -> xyz=0.20990559999999747198 0.2505455999999988137 5.8286708792820718372e-16 rpy=1.4373447656321374473e-15 4.3984744919560549052e-16 3.1415926535897922278; parent legjointconnector2_3 -> legjointconnector2_4
- joint BR_J4: child legjointconnector4_3 -> legjointconnector4_4; limit lower=0 upper=6.283185307179586232 effort=1 velocity=20 -> lower=-1.0471975511965976313 upper=0.34906585039886589561 effort=1 velocity=20; origin xyz=-1.1645024028449080244 0 -4.4408920985006261617e-16 rpy=-9.0442043540577272659e-17 -4.478155192180798781e-17 -2.5970077749655048884e-17 -> xyz=-1.1645024028448931475 -1.8873791418627661187e-15 -1.4988010832439613296e-15 rpy=-1.7655377548137906651e-15 -8.4596118181461122216e-17 2.4739660131420130417e-15; parent segment3_3 -> segment3_4
- joint FL_J1: child base -> segment1inverse; limit lower=0 upper=6.283185307179586232 effort=1 velocity=20 -> lower=-0.87266462599716476678 upper=0 effort=1 velocity=20; origin xyz=-0.57807399120160729566 -0.5988052311389459037 -0.77874950167232726006 rpy=-2.3872993578795250843e-08 3.8169197161100659601e-08 -1.5707963267948970021 -> xyz=-1.060651181194484094 -0.3720785334857630855 -0.14137121336743724287 rpy=4.13660654493550868e-08 -1.5386514143357501996e-08 0.87266463153052498125; parent segment1inverse -> base
- joint FL_J2: child legjointconnector2_4 -> legjointconnector2_2; limit lower=0 upper=6.283185307179586232 effort=1 velocity=20 -> lower=-1.3962634015954635824 upper=0.52359877559829881566 effort=1 velocity=20; origin xyz=-1.0338515942334769449 -0.32245322629145822813 -0.90574948024341750408 rpy=1.5707962886256991997 -2.3872993467772918602e-08 -3.1415926535897926719 -> xyz=-0.45577759999999967189 0.27635199999999893183 -0.12700000000000119527 rpy=1.5707963267948972241 0.52359877559828815752 -3.1415926535897926719
- joint FL_J3: child segment3_4 -> segment3_2; limit lower=0 upper=6.283185307179586232 effort=1 velocity=20 -> lower=-1.0471975511965976313 upper=0.34906585039886589561 effort=1 velocity=20; origin xyz=0.20990560000000035856 0.2505455999999998129 5.5511151231257827021e-17 rpy=4.2376321985735554229e-24 1.0729593300831567566e-17 3.141592653589793116 -> xyz=0.20990560000000013652 0.25054559999999992392 -1.1102230246251565404e-16 rpy=3.3343912457666189774e-16 -4.6147739789338615047e-15 3.1415926535897922278; parent legjointconnector2_4 -> legjointconnector2_2
- joint FL_J4: child legjointconnector4_4 -> legjointconnector4_2; limit lower=0 upper=6.3006385996995293297 effort=1 velocity=20 -> lower=-1.0471975511965976313 upper=0.34906585039886589561 effort=1 velocity=20; origin xyz=-1.1645024028449064701 -1.1102230246251565404e-16 1.1102230246251565404e-16 rpy=-1.110222826101810144e-16 -1.1778011199458197558e-30 -1.5278887872991683262e-23 -> xyz=-1.1645024028449126874 -4.4408920985006261617e-16 1.8873791418627661187e-15 rpy=-1.1469567991054151564e-15 6.4836619306514026563e-16 2.3592702349518586125e-16; parent segment3_4 -> segment3_2
- joint FR_J1: limit lower=0 upper=6.283185307179586232 effort=1 velocity=20 -> lower=0 upper=0.87266462599716476678 effort=1 velocity=20; origin xyz=0 0.96519999999999961382 0 rpy=2.9004576563626872302e-15 1.013078515305890832e-15 -1.5707963267948972241 -> xyz=-0.44023258441632540094 0.3673075664456756928 -0.14137119851637669488 rpy=-4.1366039038186796774e-08 1.538652296404905063e-08 -2.2689280220592675796
- joint FR_J2: child legjointconnector2_2 -> legjointconnector2_3; limit lower=0 upper=6.283185307179586232 effort=1 velocity=20 -> lower=-0.52359877559829881566 upper=1.3962634015954635824 effort=1 velocity=20; origin xyz=-0.4557775999999997274 -0.27635199999999998655 -0.12699999999999977973 rpy=-1.5707963267948947816 5.8286706669016316343e-16 3.141592653589793116 -> xyz=-0.45577759999999989393 -0.27635199999999915388 -0.12699999999999947442 rpy=-1.5707963267948974462 0.52359877559829615112 3.1415926535897762406
- joint FR_J3: child segment3_2 -> segment3_3; limit lower=0 upper=6.283185307179586232 effort=1 velocity=20 -> lower=-0.34906585039886589561 upper=1.0471975511965976313 effort=1 velocity=20; origin xyz=0.2099056000000000255 -0.25054559999999992392 -5.5511151231257827021e-17 rpy=5.5511156512876473097e-17 1.8316849040800762374e-31 3.141592653589793116 -> xyz=0.20990560000000024754 -0.25054560000000014597 2.2204460492503130808e-16 rpy=-1.8985674999768793355e-15 1.23596449809788972e-14 -3.141592653589763362; parent legjointconnector2_2 -> legjointconnector2_3
- joint FR_J4: child legjointconnector4_2 -> legjointconnector4_3; limit lower=0 upper=6.283185307179586232 effort=1 velocity=20 -> lower=-0.34906585039886589561 upper=1.0471975511965976313 effort=1 velocity=20; origin xyz=-1.1645024028449086906 -1.1102230246251565404e-16 1.6653345369377348106e-16 rpy=1.605866653096347499e-15 -4.3247425860249348976e-18 -4.0123531872111090802e-17 -> xyz=-1.1645024028448989206 -1.9428902930940239457e-16 9.9920072216264088638e-16 rpy=2.0702645687492304713e-15 -1.2750068319148383268e-14 -1.7893969234326057185e-16; parent segment3_2 -> segment3_3
