Commit message: absolute version

File: V2_Env_Model/Model/robot.urdf (robot description, URDF)
Before this commit: robot onshape, 17 links, 16 joints
Links:
- link base: mass 1406.2088699182118035 -> 6000.0
- link legjointconnector2: mass 33.700879238921572778 -> 200.0
- link legjointconnector2_2: mass 33.700879238921572778 -> 200.0
- link legjointconnector2_3: mass 33.700879238921572778 -> 200.0
- link legjointconnector2_4: mass 33.700879238921572778 -> 200.0
- link legjointconnector4: mass 113.67855069945755986 -> 1200.0
- link legjointconnector4_2: mass 113.67855069945755986 -> 1200.0
- link legjointconnector4_3: mass 113.67855069945755986 -> 1200.0
- link legjointconnector4_4: mass 113.67855069945755986 -> 1200.0
- link segment1: mass 188.73631876709129074 -> 800.0
- link segment1_2: mass 188.73631876709129074 -> 800.0
- link segment1inverse: mass 188.73631876709129074 -> 800.0
- link segment1inverse_2: mass 188.73631876709129074 -> 800.0
- link segment3: mass 415.11154881410027429 -> 1600
- link segment3_2: mass 415.11154881410027429 -> 1600
- link segment3_3: mass 415.11154881410027429 -> 1600
- link segment3_4: mass 415.11154881410027429 -> 1600
Joints:
- joint BL_J1: limit lower=0 upper=0.87266462599716476678 effort=1 velocity=20 -> lower=0 upper=0.87266462599716476678 velocity=20
- joint BL_J2: limit lower=-0.52359877559829881566 upper=1.3962634015954635824 effort=1 velocity=20 -> lower=-0.52359877559829881566 upper=1.3962634015954635824 velocity=20
- joint BL_J3: limit lower=-0.34906585039886589561 upper=1.0471975511965976313 effort=1 velocity=20 -> lower=-0.34906585039886589561 upper=1.0471975511965976313 velocity=20
- joint BL_J4: limit lower=-0.34906585039886589561 upper=1.0471975511965976313 effort=1 velocity=20 -> lower=-0.34906585039886589561 upper=1.0471975511965976313 velocity=20
- joint BR_J1: limit lower=-0.87266462599716476678 upper=0 effort=1 velocity=20 -> lower=-0.87266462599716476678 upper=0 velocity=20
- joint BR_J2: limit lower=-1.3962634015954635824 upper=0.52359877559829881566 effort=1 velocity=20 -> lower=-1.3962634015954635824 upper=0.52359877559829881566 velocity=20
- joint BR_J3: limit lower=-1.0471975511965976313 upper=0.34906585039886589561 effort=1 velocity=20 -> lower=-1.0471975511965976313 upper=0.34906585039886589561 velocity=20
- joint BR_J4: limit lower=-1.0471975511965976313 upper=0.34906585039886589561 effort=1 velocity=20 -> lower=-1.0471975511965976313 upper=0.34906585039886589561 velocity=20
- joint FL_J1: limit lower=-0.87266462599716476678 upper=0 effort=1 velocity=20 -> lower=-0.87266462599716476678 upper=0 velocity=20
- joint FL_J2: limit lower=-1.3962634015954635824 upper=0.52359877559829881566 effort=1 velocity=20 -> lower=-1.3962634015954635824 upper=0.52359877559829881566 velocity=20
- joint FL_J3: limit lower=-1.0471975511965976313 upper=0.34906585039886589561 effort=1 velocity=20 -> lower=-1.0471975511965976313 upper=0.34906585039886589561 velocity=20
- joint FL_J4: limit lower=-1.0471975511965976313 upper=0.34906585039886589561 effort=1 velocity=20 -> lower=-1.0471975511965976313 upper=0.34906585039886589561 velocity=20
- joint FR_J1: limit lower=0 upper=0.87266462599716476678 effort=1 velocity=20 -> lower=0 upper=0.87266462599716476678 velocity=20
- joint FR_J2: limit lower=-0.52359877559829881566 upper=1.3962634015954635824 effort=1 velocity=20 -> lower=-0.52359877559829881566 upper=1.3962634015954635824 velocity=20
- joint FR_J3: limit lower=-0.34906585039886589561 upper=1.0471975511965976313 effort=1 velocity=20 -> lower=-0.34906585039886589561 upper=1.0471975511965976313 velocity=20
- joint FR_J4: limit lower=-0.34906585039886589561 upper=1.0471975511965976313 effort=1 velocity=20 -> lower=-0.34906585039886589561 upper=1.0471975511965976313 velocity=20

Commit message: reduce vel, multi-env training

File: V2_Env_Model/Model/robot.urdf (robot description, URDF)
Before this commit: robot onshape, 17 links, 16 joints
Links:
- link base: mass 6000.0 -> 1406.2088699182118035
- link legjointconnector2: mass 200.0 -> 33.700879238921572778
- link legjointconnector2_2: mass 200.0 -> 33.700879238921572778
- link legjointconnector2_3: mass 200.0 -> 33.700879238921572778
- link legjointconnector2_4: mass 200.0 -> 33.700879238921572778
- link legjointconnector4: mass 1200.0 -> 113.67855069945755986
- link legjointconnector4_2: mass 1200.0 -> 113.67855069945755986
- link legjointconnector4_3: mass 1200.0 -> 113.67855069945755986
- link legjointconnector4_4: mass 1200.0 -> 113.67855069945755986
- link segment1: mass 800.0 -> 188.73631876709129074
- link segment1_2: mass 800.0 -> 188.73631876709129074
- link segment1inverse: mass 800.0 -> 188.73631876709129074
- link segment1inverse_2: mass 800.0 -> 188.73631876709129074
- link segment3: mass 1600 -> 415.11154881410027429
- link segment3_2: mass 1600 -> 415.11154881410027429
- link segment3_3: mass 1600 -> 415.11154881410027429
- link segment3_4: mass 1600 -> 415.11154881410027429
Joints:
- joint BL_J1: limit lower=0 upper=0.87266462599716476678 velocity=20 -> lower=0 upper=0.87266462599716476678 effort=1 velocity=10
- joint BL_J2: limit lower=-0.52359877559829881566 upper=1.3962634015954635824 velocity=20 -> lower=-0.52359877559829881566 upper=1.3962634015954635824 effort=1 velocity=10
- joint BL_J3: limit lower=-0.34906585039886589561 upper=1.0471975511965976313 velocity=20 -> lower=-0.34906585039886589561 upper=1.0471975511965976313 effort=1 velocity=10
- joint BL_J4: limit lower=-0.34906585039886589561 upper=1.0471975511965976313 velocity=20 -> lower=-0.34906585039886589561 upper=1.0471975511965976313 effort=1 velocity=10
- joint BR_J1: limit lower=-0.87266462599716476678 upper=0 velocity=20 -> lower=-0.87266462599716476678 upper=0 effort=1 velocity=10
- joint BR_J2: limit lower=-1.3962634015954635824 upper=0.52359877559829881566 velocity=20 -> lower=-1.3962634015954635824 upper=0.52359877559829881566 effort=1 velocity=10
- joint BR_J3: limit lower=-1.0471975511965976313 upper=0.34906585039886589561 velocity=20 -> lower=-1.0471975511965976313 upper=0.34906585039886589561 effort=1 velocity=10
- joint BR_J4: limit lower=-1.0471975511965976313 upper=0.34906585039886589561 velocity=20 -> lower=-1.0471975511965976313 upper=0.34906585039886589561 effort=1 velocity=10
- joint FL_J1: limit lower=-0.87266462599716476678 upper=0 velocity=20 -> lower=-0.87266462599716476678 upper=0 effort=1 velocity=10
- joint FL_J2: limit lower=-1.3962634015954635824 upper=0.52359877559829881566 velocity=20 -> lower=-1.3962634015954635824 upper=0.52359877559829881566 effort=1 velocity=10
- joint FL_J3: limit lower=-1.0471975511965976313 upper=0.34906585039886589561 velocity=20 -> lower=-1.0471975511965976313 upper=0.34906585039886589561 effort=1 velocity=10
- joint FL_J4: limit lower=-1.0471975511965976313 upper=0.34906585039886589561 velocity=20 -> lower=-1.0471975511965976313 upper=0.34906585039886589561 effort=1 velocity=10
- joint FR_J1: limit lower=0 upper=0.87266462599716476678 velocity=20 -> lower=0 upper=0.87266462599716476678 effort=1 velocity=10
- joint FR_J2: limit lower=-0.52359877559829881566 upper=1.3962634015954635824 velocity=20 -> lower=-0.52359877559829881566 upper=1.3962634015954635824 effort=1 velocity=10
- joint FR_J3: limit lower=-0.34906585039886589561 upper=1.0471975511965976313 velocity=20 -> lower=-0.34906585039886589561 upper=1.0471975511965976313 effort=1 velocity=10
- joint FR_J4: limit lower=-0.34906585039886589561 upper=1.0471975511965976313 velocity=20 -> lower=-0.34906585039886589561 upper=1.0471975511965976313 effort=1 velocity=10

Commit message: network depth increase

File: V2_Env_Model/Model/robot.urdf (robot description, URDF)
Before this commit: robot onshape, 17 links, 16 joints
Links:
- link base: mass 1406.2088699182118035 -> 1406.2088699182113487
- link legjointconnector4: mass 113.67855069945755986 -> 113.67855069945754565
- link legjointconnector4_2: mass 113.67855069945755986 -> 113.67855069945754565
- link legjointconnector4_3: mass 113.67855069945755986 -> 113.67855069945754565
- link legjointconnector4_4: mass 113.67855069945755986 -> 113.67855069945754565
Joints:
- joint BL_J1: limit lower=0 upper=0.87266462599716476678 effort=1 velocity=10 -> lower=0 upper=0.87266462599716476678 effort=1 velocity=20
- joint BL_J2: limit lower=-0.52359877559829881566 upper=1.3962634015954635824 effort=1 velocity=10 -> lower=-0.52359877559829881566 upper=1.3962634015954635824 effort=1 velocity=20
- joint BL_J3: limit lower=-0.34906585039886589561 upper=1.0471975511965976313 effort=1 velocity=10 -> lower=-0.34906585039886589561 upper=0.34906585039886589561 effort=1 velocity=20
- joint BL_J4: limit lower=-0.34906585039886589561 upper=1.0471975511965976313 effort=1 velocity=10 -> lower=-0.34906585039886589561 upper=1.0471975511965976313 effort=1 velocity=20
- joint BR_J1: limit lower=-0.87266462599716476678 upper=0 effort=1 velocity=10 -> lower=-0.87266462599716476678 upper=0 effort=1 velocity=20
- joint BR_J2: limit lower=-1.3962634015954635824 upper=0.52359877559829881566 effort=1 velocity=10 -> lower=-1.3962634015954635824 upper=0.52359877559829881566 effort=1 velocity=20
- joint BR_J3: limit lower=-1.0471975511965976313 upper=0.34906585039886589561 effort=1 velocity=10 -> lower=-0.34906585039886589561 upper=0.34906585039886589561 effort=1 velocity=20
- joint BR_J4: limit lower=-1.0471975511965976313 upper=0.34906585039886589561 effort=1 velocity=10 -> lower=-1.0471975511965976313 upper=0.34906585039886589561 effort=1 velocity=20
- joint FL_J1: limit lower=-0.87266462599716476678 upper=0 effort=1 velocity=10 -> lower=-0.87266462599716476678 upper=0 effort=1 velocity=20
- joint FL_J2: limit lower=-1.3962634015954635824 upper=0.52359877559829881566 effort=1 velocity=10 -> lower=-1.3962634015954635824 upper=0.52359877559829881566 effort=1 velocity=20
- joint FL_J3: limit lower=-1.0471975511965976313 upper=0.34906585039886589561 effort=1 velocity=10 -> lower=-0.34906585039886589561 upper=0.34906585039886589561 effort=1 velocity=20
- joint FL_J4: limit lower=-1.0471975511965976313 upper=0.34906585039886589561 effort=1 velocity=10 -> lower=-1.0471975511965976313 upper=0.34906585039886589561 effort=1 velocity=20
- joint FR_J1: limit lower=0 upper=0.87266462599716476678 effort=1 velocity=10 -> lower=0 upper=0.87266462599716476678 effort=1 velocity=20
- joint FR_J2: limit lower=-0.52359877559829881566 upper=1.3962634015954635824 effort=1 velocity=10 -> lower=-0.52359877559829881566 upper=1.3962634015954635824 effort=1 velocity=20
- joint FR_J3: limit lower=-0.34906585039886589561 upper=1.0471975511965976313 effort=1 velocity=10 -> lower=-0.34906585039886589561 upper=0.34906585039886589561 effort=1 velocity=20
- joint FR_J4: limit lower=-0.34906585039886589561 upper=1.0471975511965976313 effort=1 velocity=10 -> lower=-0.34906585039886589561 upper=1.0471975511965976313 effort=1 velocity=20
