Commit message: hard code with turn

File: V3_Env_Model/Model/robot.urdf (robot description, URDF)
Before this commit: robot onshape, 17 links, 16 joints
Joints:
- joint BL_J3: limit lower=-0.1745329251994329478 upper=0.1745329251994329478 effort=1 velocity=20 -> lower=-0.34906585039886589561 upper=0.34906585039886589561 effort=1 velocity=20
- joint BR_J3: limit lower=-0.1745329251994329478 upper=0.1745329251994329478 effort=1 velocity=20 -> lower=-0.34906585039886589561 upper=0.34906585039886589561 effort=1 velocity=20
- joint FL_J3: limit lower=-0.1745329251994329478 upper=0.1745329251994329478 effort=1 velocity=20 -> lower=-0.34906585039886589561 upper=0.34906585039886589561 effort=1 velocity=20
- joint FR_J3: limit lower=-0.1745329251994329478 upper=0.1745329251994329478 effort=1 velocity=20 -> lower=-0.34906585039886589561 upper=0.34906585039886589561 effort=1 velocity=20

Commit message: hardcoded gait, auto-alignment

File: V3_Env_Model/Model/robot.urdf (robot description, URDF)
Before this commit: robot onshape, 17 links, 16 joints
Links:
- link base: mass 1406.2088699182113487 -> 1406.2088699182118035
- link legjointconnector2: mass 33.700879238921558567 -> 33.700879238921572778
- link legjointconnector2_2: mass 33.700879238921558567 -> 33.700879238921572778
- link legjointconnector2_3: mass 33.700879238921558567 -> 33.700879238921572778
- link legjointconnector2_4: mass 33.700879238921558567 -> 33.700879238921572778
- link legjointconnector4: mass 113.67855069945754565 -> 113.67855069945751723
- link legjointconnector4_2: mass 113.67855069945754565 -> 113.67855069945751723
- link legjointconnector4_3: mass 113.67855069945754565 -> 113.67855069945751723
- link legjointconnector4_4: mass 113.67855069945754565 -> 113.67855069945751723
Joints:
- joint BL_J2: origin xyz=-0.45577759999999978291 -0.27635199999999915388 -0.12699999999999922462 rpy=-1.570796326794896336 -1.1133486160753729077e-16 -3.1415926535897860106 -> xyz=-0.45577759999999956086 -0.27635199999999870979 -0.12699999999999922462 rpy=-1.570796326794896336 -5.5823697141391807618e-17 -3.1415926535897860106
- joint BL_J3: limit lower=-0.34906585039886589561 upper=0.34906585039886589561 effort=1 velocity=20 -> lower=-0.1745329251994329478 upper=0.1745329251994329478 effort=1 velocity=20; origin xyz=0.20990560000000035856 -0.25054559999999992392 0 rpy=-2.5283167277087328215e-15 3.1919323348587798512e-15 3.1415926535897922278 -> xyz=0.20990560000000035856 -0.25054559999999992392 -5.5511151231257827021e-17 rpy=4.0009830263683715674e-15 3.7623924145558519288e-15 3.1415926535897891192
- joint BL_J4: origin xyz=-1.1645024028449160181 -1.3877787807814456755e-17 9.7144514654701197287e-15 rpy=-1.0002491849452616732e-14 -1.8279819730990857957e-14 2.5535131700721312462e-15 -> xyz=-1.1645024028449084685 -3.1086244689504383132e-15 1.7208456881689926377e-15 rpy=-1.4753334857957956014e-15 1.7721323323395540624e-16 4.218851918506896105e-15
- joint BR_J2: origin xyz=-0.45577759999999961638 0.27635199999999998655 -0.12699999999999997402 rpy=1.570796326794896336 -1.4139325538541093417e-14 3.1415926535897926719 -> xyz=-0.45577759999999961638 0.27635199999999993103 -0.12699999999999991851 rpy=1.570796326794896336 2.5617351588273872295e-15 -3.1415926535897726879
- joint BR_J3: limit lower=-0.34906585039886589561 upper=0.34906585039886589561 effort=1 velocity=20 -> lower=-0.1745329251994329478 upper=0.1745329251994329478 effort=1 velocity=20; origin xyz=0.20990560000000008101 0.25054559999999992392 -5.5511151231257827021e-17 rpy=-7.143255743244556814e-17 -7.0098970658315433197e-16 3.1415926535897775729 -> xyz=0.2099056000000000255 0.25054559999999997943 -1.1102230246251565404e-16 rpy=-2.4583537112042395624e-14 1.7733630015494619918e-14 3.1415926535897771288
- joint BR_J4: origin xyz=-1.1645024028449151299 7.8409501114151680667e-16 -7.5495165674510644749e-15 rpy=-1.8770539177431924915e-15 6.4170359308439466523e-16 -2.2204497208545383792e-16 -> xyz=-1.1645024028449117992 -3.8163916471489756077e-17 -3.1363800445660672267e-14 rpy=1.1607104557275275595e-14 -1.317684822795214061e-14 1.7097434238094243648e-14
- joint FL_J2: origin xyz=-0.45577759999999978291 0.27635199999999837672 -0.12699999999999925238 rpy=1.570796326794896336 8.4958856427445189586e-15 3.1415926535897917837 -> xyz=-0.45577759999999978291 0.27635199999999815468 -0.12699999999999930789 rpy=1.570796326794896336 -1.6817628903380697032e-14 3.1415926535897527039
- joint FL_J3: limit lower=-0.34906585039886589561 upper=0.34906585039886589561 effort=1 velocity=20 -> lower=-0.1745329251994329478 upper=0.1745329251994329478 effort=1 velocity=20; origin xyz=0.20990560000000035856 0.25054559999999992392 0 rpy=1.0838683866018271256e-15 -4.2368862056886156146e-15 -3.1415926535897842342 -> xyz=0.20990560000000169083 0.25054560000000120068 -8.2156503822261583991e-15 rpy=1.6194871490508681314e-15 -4.0628214769688119786e-14 3.1415926535897766847
- joint FL_J4: origin xyz=-1.1645024028448953679 -7.9797279894933126343e-17 -1.9984014443252817728e-15 rpy=-1.4230303722337115841e-14 1.0989215082908320336e-14 -1.9142660398205388481e-22 -> xyz=-1.1645024028449084685 -6.5919492087118669588e-17 -8.8817841970012523234e-16 rpy=-5.3187625266587315242e-16 2.223579799404422412e-15 -9.1593406069752589358e-15
- joint FR_J2: origin xyz=-0.45577759999999978291 -0.27635199999999360276 -0.12700000000000097322 rpy=-1.570796326794896336 -1.1199904040369779026e-14 -3.1415926535897868987 -> xyz=-0.45577759999999983842 -0.27635200000000093024 -0.12700000000000108424 rpy=-1.570796326794896336 -5.0898889851839357653e-14 3.1415926535897900074
- joint FR_J3: limit lower=-0.34906585039886589561 upper=0.34906585039886589561 effort=1 velocity=20 -> lower=-0.1745329251994329478 upper=0.1745329251994329478 effort=1 velocity=20; origin xyz=0.20990560000000035856 -0.25054559999999992392 0 rpy=1.1168225010396418927e-14 6.9265645206730398148e-15 -3.1415926535897149563 -> xyz=0.20990560000000030305 -0.25054559999999997943 -2.2204460492503130808e-16 rpy=1.8312212865081671257e-15 1.0372016758782980754e-15 -3.1415926535897047422
- joint FR_J4: origin xyz=-1.164502402844935558 -3.1225022567582527699e-17 4.4408920985006261617e-16 rpy=-3.8581974629149813854e-14 -2.1207345775403515895e-14 -7.3163696734599736933e-14 -> xyz=-1.1645024028449388886 1.1449174941446926823e-16 2.2204460492503130808e-16 rpy=-6.2303374567070360012e-14 -7.5210931242245077766e-14 -4.7239990430088080467e-14
